File: Project Architecture.kicad_sch (KiCad schematic)
At the start: 0 parts

Commit message: First draft of the schematic
Other:
- sheet Section A - Title A renamed MCU
- sheet Section B - Title B renamed IMU
Changed lines of the file:
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@@
 (kicad_sch
-	(version 20231120)
+	(version 20250114)
 	(generator "eeschema")
-	(generator_version "8.0")
+	(generator_version "9.0")
 	(paper "A3")
 	(title_block
@@
 		(company "${COMPANY}")
 	)
-	(polyline
-		(pts
-			(xy 185.42 87.63) (xy 185.42 99.06)
-		)
-		(stroke
-			(width 0)
-			(type default)
-		)
-	)
-	(polyline
-		(pts
-			(xy 233.68 125.73) (xy 233.68 134.62)
-		)
-		(stroke
-			(width 0)
-			(type default)
-		)
-	)
-	(polyline
-		(pts
-			(xy 185.42 85.09) (xy 185.42 73.66)
-		)
-		(stroke
-			(width 0)
-			(type default)
-		)
-	)
-	(polyline
-		(pts
-			(xy 233.68 114.3) (xy 233.68 123.19)
-		)
-		(stroke
-			(width 0)
-			(type default)
-		)
-	)
 	(arc
 		(start 185.42 85.09)
@@
 	)
 	(arc
-		(start 234.97 124.44)
-		(mid 234.0749 124.0651)
-		(end 233.7 123.17)
-		(stroke
-			(width 0)
-			(type default)
-		)
-		(fill
-			(type none)
-		)
-	)
-	(arc
-		(start 233.7 125.71)
-		(mid 234.0749 124.8149)
-		(end 234.97 124.44)
-		(stroke
-			(width 0)
-			(type default)
-		)
-		(fill
-			(type none)
-		)
-	)
-	(arc
-		(start 233.7 134.6)
-		(mid 232.9561 136.3961)
-		(end 231.16 137.14)
+		(start 284.5 86.34)
+		(mid 283.6049 85.9651)
+		(end 283.23 85.07)
+		(stroke
+			(width 0)
+			(type default)
+		)
+		(fill
+			(type none)
+		)
+	)
+	(arc
+		(start 283.23 87.61)
+		(mid 283.6049 86.7149)
+		(end 284.5 86.34)
+		(stroke
+			(width 0)
+			(type default)
+		)
+		(fill
+			(type none)
+		)
+	)
+	(arc
+		(start 283.23 96.5)
+		(mid 282.4861 98.2961)
+		(end 280.69 99.04)
 		(stroke
 			(width 0)
@@
 	)
 	(arc
-		(start 231.16 111.74)
-		(mid 232.9502 112.4898)
-		(end 233.7 114.28)
+		(start 280.69 73.64)
+		(mid 282.4802 74.3898)
+		(end 283.23 76.18)
 		(stroke
 			(width 0)
@@
 		)
 	)
+	(text "Page 5"
+		(exclude_from_sim no)
+		(at 275.59 95.25 0)
+		(effects
+			(font
+				(size 2.54 2.54)
+				(bold yes)
+				(color 100 70 50 1)
+			)
+			(justify right bottom)
+			(href "#5")
+		)
+	)
+	(text "Page 4"
+		(exclude_from_sim no)
+		(at 226.06 95.25 0)
+		(effects
+			(font
+				(size 2.54 2.54)
+				(bold yes)
+				(color 20 60 40 1)
+			)
+			(justify right bottom)
+			(href "#4")
+		)
+	)
 	(text_box "Description"
 		(exclude_from_sim no)
 		(at 166.37 83.82 0)
 		(size 17.145 5.08)
+		(margins 1.4287 1.4287 1.4287 1.4287)
 		(stroke
 			(width -0.0001)
@@
 	(text_box "Description"
 		(exclude_from_sim no)
-		(at 234.95 121.92 0)
+		(at 284.48 83.82 0)
 		(size 26.015 5.1)
+		(margins 1.4287 1.4287 1.4287 1.4287)
 		(stroke
 			(width -0.0001)
@@
 		(at 144.78 21.59 0)
 		(size 130.81 12.7)
+		(margins 5.9999 5.9999 5.9999 5.9999)
 		(stroke
 			(width -0.0001)
@@
 		)
 	)
-	(text "Page 5"
-		(exclude_from_sim no)
-		(at 226.06 133.35 0)
-		(effects
-			(font
-				(size 2.54 2.54)
-				(bold yes)
-				(color 100 70 50 1)
-			)
-			(justify right bottom)
-			(href "#5")
-		)
-	)
-	(text "Page 4"
-		(exclude_from_sim no)
-		(at 226.06 95.25 0)
-		(effects
-			(font
-				(size 2.54 2.54)
-				(bold yes)
-				(color 20 60 40 1)
-			)
-			(justify right bottom)
-			(href "#4")
+	(polyline
+		(pts
+			(xy 240.03 85.09) (xy 240.03 86.36)
+		)
+		(stroke
+			(width 0)
+			(type default)
+		)
+	)
+	(polyline
+		(pts
+			(xy 185.42 87.63) (xy 185.42 99.06)
+		)
+		(stroke
+			(width 0)
+			(type default)
+		)
+	)
+	(polyline
+		(pts
+			(xy 283.21 87.63) (xy 283.21 96.52)
+		)
+		(stroke
+			(width 0)
+			(type default)
+		)
+	)
+	(polyline
+		(pts
+			(xy 185.42 85.09) (xy 185.42 73.66)
+		)
+		(stroke
+			(width 0)
+			(type default)
+		)
+	)
+	(polyline
+		(pts
+			(xy 283.21 76.2) (xy 283.21 85.09)
+		)
+		(stroke
+			(width 0)
+			(type default)
+		)
+	)
+	(bus
+		(pts
+			(xy 227.33 86.36) (xy 240.03 86.36)
+		)
+		(stroke
+			(width 0)
+			(type default)
+		)
+	)
+	(hierarchical_label "{SPI1}"
+		(shape bidirectional)
+		(at 240.03 86.36 0)
+		(effects
+			(font
+				(size 1.27 1.27)
+			)
+			(justify left)
+		)
+	)
+	(hierarchical_label "{SPI1}"
+		(shape bidirectional)
+		(at 227.33 86.36 180)
+		(effects
+			(font
+				(size 1.27 1.27)
+			)
+			(justify right)
 		)
 	)
 	(sheet
-		(at 190.5 114.3)
+		(at 240.03 76.2)
 		(size 36.83 20.32)
+		(exclude_from_sim no)
+		(in_bom yes)
+		(on_board yes)
+		(dnp no)
 		(fields_autoplaced yes)
 		(stroke
@@
 			(color 255 200 0 0.5020)
 		)
-		(property "Sheetname" "Section B - Title B"
-			(at 190.5 113.2709 0)
+		(property "Sheetname" "IMU"
+			(at 240.03 75.1709 0)
 			(effects
 				(font
@@
 		)
 		(property "Sheetfile" "Section B - TItle B.kicad_sch"
-			(at 190.5 135.2046 0)
+			(at 240.03 97.1046 0)
 			(effects
 				(font
@@
 		)
 		(instances
-			(project "KDT_Hierarchical_KiBot"
+			(project "seismic_sensor"
 				(path "/f9e05184-c88b-4a88-ae9c-ab2bdb32be7c/c5103ceb-5325-4a84-a025-9638a412984e"
 					(page "5")
@@
 		(at 190.5 76.2)
 		(size 36.83 20.32)
+		(exclude_from_sim no)
+		(in_bom yes)
+		(on_board yes)
+		(dnp no)
 		(fields_autoplaced yes)
 		(stroke
@@
 			(color 128 255 128 0.5000)
 		)
-		(property "Sheetname" "Section A - Title A"
+		(property "Sheetname" "MCU"
 			(at 190.5 75.1709 0)
 			(effects
@@
 		)
 		(instances
-			(project "KDT_Hierarchical_KiBot"
+			(project "seismic_sensor"
 				(path "/f9e05184-c88b-4a88-ae9c-ab2bdb32be7c/c5103ceb-5325-4a84-a025-9638a412984e"
 					(page "4")
