File: Section B - TItle B.kicad_sch (KiCad schematic)
At the start: 0 parts

Commit message: First draft of the schematic
Parts:
- added C1: 0.1uF, symbol Device:C
- added C2: 10uF, symbol Device:C
- added FB1: FerriteBead, symbol Device:FerriteBead
- added U2: ADXL345BCCZ, LGA_CC-14-1_ADI, symbol 2026-02-02_16-19-33:ADXL345BCCZ
Connections:
- new net: FB1.2, U2.6 (VS)
- new net +3V3: C1.1, C2.1, FB1.1, U2.1 (VDD_I/O)
- new net CS*: U2.7 (*CS)
- new net GND: C1.2, C2.2, U2.2 (GND), U2.4 (GND), U2.5 (GND)
- new net SCLK: U2.14 (SCL/SCLK)
- new net SDI: U2.13 (SDA/SDI/SDIO)
- new net SDO: U2.12 (SDO/ALT_ADDRESS)
- no-connect marks 0 -> 3
