File: Block Diagram.kicad_sch (KiCad schematic)
At the start: 0 parts

Commit message: updated structure
Other:
- note added: "+3.3V"
- note added: "2.6V - 4.3V"
Changed lines of the file:
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@@
+		)
+	)
+	(text "2.6V - 4.3V"
+		(exclude_from_sim no)
+		(at 45.212 76.2 0)
+		(effects
+			(font
+				(face "Times New Roman")
+				(size 2.286 2.286)
+				(thickness 0.4572)
+				(bold yes)
+				(color 0 0 0 1)
+			)
+			(justify left bottom)
+		)
+	)
+	(text "+3.3V"
+		(exclude_from_sim no)
+		(at 129.54 76.2 0)
+		(effects
+			(font
+				(face "Times New Roman")
+				(size 2.286 2.286)
+				(thickness 0.4572)
+				(bold yes)
+				(color 0 0 0 1)
+			)
+			(justify left bottom)
+		)
+	)
+	(text "+A3V3"
+		(exclude_from_sim no)
+		(at 130.81 109.22 0)
+		(effects
+			(font
+				(face "Times New Roman")
+				(size 2.286 2.286)
+				(thickness 0.4572)
+				(bold yes)
+				(color 0 0 0 1)
+			)
+			(justify left bottom)
 		)
 	)
 	(text "+??V"
 		(exclude_from_sim no)
-		(at 49.53 76.2 0)
-		(effects
-			(font
-				(face "Times New Roman")
-				(size 2.286 2.286)
-				(thickness 0.4572)
-				(bold yes)
-				(color 0 0 0 1)
-			)
-			(justify left bottom)
-		)
-	)
-	(text "+??V"
-		(exclude_from_sim no)
-		(at 129.54 76.2 0)
-		(effects
-			(font
-				(face "Times New Roman")
-				(size 2.286 2.286)
-				(thickness 0.4572)
-				(bold yes)
-				(color 0 0 0 1)
-			)
-			(justify left bottom)
-		)
-	)
-	(text "+A3V3"
-		(exclude_from_sim no)
-		(at 130.81 109.22 0)
-		(effects
-			(font
-				(face "Times New Roman")
-				(size 2.286 2.286)
-				(thickness 0.4572)
-				(bold yes)
-				(color 0 0 0 1)
-			)
-			(justify left bottom)
-		)
-	)
-	(text "+??V"
-		(exclude_from_sim no)
 		(at 119.38 95.25 0)
 		(effects
@@
 		)
 	)
-	(text "+??V"
+	(text "+3.3V"
 		(exclude_from_sim no)
 		(at 120.65 76.2 0)
@@
 		)
 	)
-	(text_box "Block\nDescription"
+	(text_box "Buck-Boost Converter"
 		(exclude_from_sim no)
 		(at 73.66 82.55 0)
@@
 		(stroke
 			(width -0.0001)
-			(type default)
+			(type solid)
 		)
 		(fill
@@
 		)
 	)
-	(text_box "Page #"
+	(text_box "Page 6"
 		(exclude_from_sim no)
 		(at 62.23 66.04 0)
@@
 		(stroke
 			(width -0.0001)
-			(type default)
-		)
-		(fill
+			(type solid)
+		)
+		(fill
