File: Connectors.kicad_sch (KiCad schematic)
At the start: 7 parts, among them J1 Conn_01x02, J2 Conn_01x05, U3 TPS631012YBGR

Commit message: updated structure
Parts:
- removed C11: 22u, CAP_226ME15D_MUR, symbol 2026-02-10_14-40-51:GRM187R61A226ME15D
- removed C12: 47u, CAP_GRM216R_2X1P25_MUR, symbol 2026-02-10_14-38-14:GRM219R60J476ME44D
- removed L1: 1u, HTEK20161T-1R0MSR_CYN, symbol 2026-02-10_14-30-14:HTEK20161T-1R0MSR
- added C11: 22u, 0_capacitor_SMD:C_0603_1608Metric, symbol Device:C
- added C12: 47u, 0_capacitor_SMD:C_0805_2012Metric, symbol Device:C
- added L2: 1u, 0_inductor:HTEK20161T-1R0MSR_CYN, symbol Device:L
- C10: footprint (none) -> 0_capacitor_SMD:C_0402_1005Metric; Manufacturer (none) -> KEMET; Manufacturer Part Number (none) -> C0402C104K8RAC
- J1: footprint Connector_JST:JST_EH_B2B-EH-A_1x02_P2.50mm_Vertical -> 0_connectors:JST_EH_B2B-EH-A_1x02_P2.50mm_Vertical
- J2: footprint (none) -> 0_connectors:JST_EH_B5B-EH-A_1x05_P2.50mm_Vertical
- U3: footprint DSBGA8-YBG_TEX -> 0_switching_regulator:DSBGA8-YBG_TEX; symbol 2026-02-05_12-13-47:TPS631012YBGR -> 0_switching_regulator:TPS631012YBGR
Connections:
- net +3V3: now also C12.1
- net GND: now also C11.2, C12.2
- net VBUS: now also C11.1
- new net: L2.1, U3. (GND)
- new net: L2.2, U3. (GND)
Other:
- company: (none) -> ${COMPANY}
- title: (none) -> Connectors
