File: IMU.kicad_sch (KiCad schematic)
At the start: 4 parts, among them U2 ADXL345BCCZ

Commit message: Schematic work & cleanup
Connections:
- net CS*: no longer U2.7 (*CS)
- net INT: now reaches U2.8 (INT1)
Other:
- moved on the sheet: C1, C2, FB1

Commit message: updated structure
Parts:
- removed U2: ADXL345BCCZ, LGA_CC-14-1_ADI, symbol 2026-02-02_16-19-33:ADXL345BCCZ
- added U1: ADXL345BCCZ, 0_imu:LGA_CC-14-1_ADI, symbol 0_imu:ADXL345BCCZ
- C1: value 0.1uF -> 0.1u; footprint (none) -> 0_capacitor_SMD:C_0402_1005Metric; Manufacturer (none) -> KEMET; Manufacturer Part Number (none) -> C0402C104K8RAC
- C2: value 10uF -> 10u; footprint (none) -> 0_capacitor_SMD:C_0603_1608Metric; Manufacturer (none) -> Samsung; Manufacturer Part Number (none) -> CL10A106KP8NNNC
- FB1: footprint (none) -> 0_ferrite_beads:FB_0603_1608Metric; Manufacturer (none) -> TDK; Manufacturer Part Number (none) -> MPZ1608Y101BTD25
Connections:
- net +3V3: now also U1.1 (VDD_I/O)
- net CS*: now also U1.7 (*CS)
- net GND: now also U1.2 (GND), U1.4 (GND), U1.5 (GND)
- net INT: now also U1.8 (INT1)
- net SCLK: now also U1.14 (SCL/SCLK)
- net SDI: now also U1.13 (SDA/SDI/SDIO)
- net SDO: now also U1.12 (SDO/ALT_ADDRESS)
- net at FB1.2: now also U1.6 (VS)
Other:
- title: Sheet Title B -> IMU
- moved on the sheet: C1, C2, FB1
