File: seismic_sensor.kicad_pcb (KiCad board)
At the start: 6 copper layers, 0 parts

Commit message: updated structure
Parts:
- added C1: 0.1u, 0_capacitor_SMD:C_0402_1005Metric, F.Cu at (37.1, 176.9)
- added C10: 0.1u, 0_capacitor_SMD:C_0402_1005Metric, F.Cu at (59.5, 155.1)
- added C11: 22u, 0_capacitor_SMD:C_0603_1608Metric, F.Cu at (50.7, 163.2)
- added C12: 47u, 0_capacitor_SMD:C_0805_2012Metric, F.Cu at (59.4, 153.5)
- added C2: 10u, 0_capacitor_SMD:C_0603_1608Metric, F.Cu at (35.8, 176.7)
- added C3: 10u, 0_capacitor_SMD:C_0603_1608Metric, F.Cu at (59.6, 151.2)
- added C4: 0.1u, 0_capacitor_SMD:C_0402_1005Metric, F.Cu at (62.8, 155.2)
- added C5: 0.1u, 0_capacitor_SMD:C_0402_1005Metric, F.Cu at (55.5, 166.8)
- added C6: 0.1u, 0_capacitor_SMD:C_0402_1005Metric, F.Cu at (53.2, 168.9)
- added C7: 1u, 0_capacitor_SMD:C_0603_1608Metric, F.Cu at (45.6, 169.5)
- added C8: 1u, 0_capacitor_SMD:C_0603_1608Metric, F.Cu at (44.5, 172.8)
- added C9: 0.1u, 0_capacitor_SMD:C_0402_1005Metric, F.Cu at (45.9, 172.6)
- added FB1: FerriteBead, 0_ferrite_beads:FB_0603_1608Metric, F.Cu at (36.9, 179.8)
- added FD1: Fiducial, 0_fiducials:Fiducial_1mm_Mask2mm, F.Cu at (35.2, 136.6)
- added FD2: Fiducial, 0_fiducials:Fiducial_1mm_Mask2mm, F.Cu at (37.4, 140.4)
- added FD3: Fiducial, 0_fiducials:Fiducial_1mm_Mask2mm, F.Cu at (40.9, 136.9)
- added FD4: Fiducial, 0_fiducials:Fiducial_1mm_Mask2mm, F.Cu at (40.9, 140.4)
- added FD5: Fiducial, 0_fiducials:Fiducial_1mm_Mask2mm, F.Cu at (44.5, 136.9)
- added FD6: Fiducial, 0_fiducials:Fiducial_1mm_Mask2mm, F.Cu at (44.5, 140.4)
- added H1: M3, 0_mounting_holes:MountingHole_3.2mm_M3_Pad, F.Cu at (26.4, 144.3)
- added H2: M3, 0_mounting_holes:MountingHole_3.2mm_M3_Pad, F.Cu at (25.9, 181.0)
- added H3: M3, 0_mounting_holes:MountingHole_3.2mm_M3_Pad, F.Cu at (92.5, 183.4)
- added H4: M3, 0_mounting_holes:MountingHole_3.2mm_M3_Pad, F.Cu at (90.8, 141.3)
- added J1: Conn_01x02, 0_connectors:JST_EH_B2B-EH-A_1x02_P2.50mm_Vertical, F.Cu at (46.9, 158.5)
- added J2: Conn_01x05, 0_connectors:JST_EH_B5B-EH-A_1x05_P2.50mm_Vertical, F.Cu at (54.7, 141.4)
- added L2: 1u, 0_inductor:HTEK20161T-1R0MSR_CYN, F.Cu at (65.8, 160.9)
- added R1: 4k7, 0_resistor_SMD:R_0402_1005Metric, F.Cu at (63.1, 164.1)
- added R2: 4k7, 0_resistor_SMD:R_0402_1005Metric, F.Cu at (46.8, 166.5)
- added U1: ADXL345BCCZ, 0_imu:LGA_CC-14-1_ADI, F.Cu at (39.9, 178.5)
- added U3: TPS631012YBGR, 0_switching_regulator:DSBGA8-YBG_TEX, F.Cu at (72.3, 162.2)
- added U4: STM32U031K8U6, 0_mcu:UFQFPN-32_STM, F.Cu at (49.6, 170.4)
Other:
- board text removed: "3× 120°"
